File: hardware/controle_xyz/controle_xyz.kicad_sch (KiCad schematic)
At the start: 13 parts, among them Q1 TIP41, SW1 SW_Push, SW2 SW_Push, U1 PCF8574T

Commit message: update esquematico
Connections:
- net at A4.9 (~{ENABLE}): no longer A1.26 (GPIO20)
- net at A1.1 (GPIO0): no longer A2.9 (~{ENABLE})
- net at A1.17 (GPIO13): no longer A3.9 (~{ENABLE})
Changed lines of the file:
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@@
-	(wire
-		(pts
-			(xy 134.62 54.61) (xy 134.62 134.62)
-		)
-		(stroke
-			(width 0)
-			(type default)
-		)
-	)
 	(wire
 		(pts
@@
 	(wire
 		(pts
-			(xy 250.19 67.31) (xy 256.54 67.31)
-		)
-		(stroke
-			(width 0)
-			(type default)
-		)
-	)
-	(wire
-		(pts
 			(xy 128.27 63.5) (xy 130.81 63.5)
 		)
@@
 	(wire
 		(pts
-			(xy 182.88 134.62) (xy 187.96 134.62)
-		)
-		(stroke
-			(width 0)
-			(type default)
-		)
-	)
-	(wire
-		(pts
 			(xy 231.14 114.3) (xy 255.27 114.3)
 		)
@@
 	(wire
 		(pts
-			(xy 256.54 115.57) (xy 232.41 115.57)
-		)
-		(stroke
-			(width 0)
-			(type default)
-		)
-	)
-	(wire
-		(pts
 			(xy 185.42 144.78) (xy 185.42 147.32)
 		)
@@
 	(wire
 		(pts
-			(xy 254 53.34) (xy 201.93 53.34)
+			(xy 254 53.34) (xy 194.31 53.34)
 		)
 		(stroke
@@
 	(wire
 		(pts
-			(xy 182.88 87.63) (xy 182.88 134.62)
-		)
-		(stroke
-			(width 0)
-			(type default)
-		)
-	)
-	(wire
-		(pts
 			(xy 203.2 157.48) (xy 203.2 160.02)
 		)
@@
 	(wire
 		(pts
-			(xy 134.62 134.62) (xy 140.97 134.62)
-		)
-		(stroke
-			(width 0)
-			(type default)
-		)
-	)
-	(wire
-		(pts
 			(xy 167.64 40.64) (xy 167.64 43.18)
 		)
@@
 	(wire
 		(pts
-			(xy 256.54 67.31) (xy 256.54 115.57)
-		)
-		(stroke
-			(width 0)
-			(type default)
-		)
-	)
-	(wire
-		(pts
 			(xy 107.95 76.2) (xy 106.68 76.2)
 		)
@@
 	(wire
 		(pts
-			(xy 201.93 53.34) (xy 201.93 62.23)
+			(xy 194.31 53.34) (xy 194.31 62.23)
 		)
 		(stroke
@@
 	(wire
 		(pts
-			(xy 232.41 115.57) (xy 232.41 134.62)
-		)
-		(stroke
-			(width 0)
-			(type default)
-		)
-	)
-	(wire
-		(pts
 			(xy 151.13 119.38) (xy 151.13 118.11)
 		)
@@
 	(wire
 		(pts
-			(xy 204.47 54.61) (xy 134.62 54.61)
-		)
-		(stroke
-			(width 0)
-			(type default)
-		)
-	)
-	(wire
-		(pts
 			(xy 255.27 69.85) (xy 250.19 69.85)
 		)
@@
 	(wire
 		(pts
-			(xy 232.41 134.62) (xy 237.49 134.62)
-		)
-		(stroke
-			(width 0)
-			(type default)
-		)
-	)
-	(wire
-		(pts
 			(xy 194.31 77.47) (xy 194.31 81.28)
 		)
@@
 	(wire
 		(pts
-			(xy 204.47 87.63) (xy 182.88 87.63)
-		)
-		(stroke
-			(width 0)
-			(type default)
-		)
-	)
-	(wire
-		(pts
 			(xy 72.39 86.36) (xy 68.58 86.36)
 		)
@@
 	(wire
 		(pts
-			(xy 201.93 62.23) (xy 204.47 62.23)
-		)
-		(stroke
+			(xy 194.31 62.23) (xy 204.47 62.23)
+		)
+		(stroke
