File: hardware/controle_xyz - PCB/controle_xyz.kicad_pcb (KiCad board)
At the start: 2 copper layers, 1 part

Commit message: update kicad prj
Parts:
- added BZ1: Buzzer, Buzzer_Beeper:Buzzer_12x9.5RM7.6, F.Cu at (86.7, 122.1)
- added J1: TB007-508-03BE, TerminalBlock_CUI:TerminalBlock_CUI_TB007-508-03_1x03_P5.08mm_Horizontal, F.Cu at (52.3, 42.0)
- added J10: TB007-508-03BE, TerminalBlock_CUI:TerminalBlock_CUI_TB007-508-03_1x03_P5.08mm_Horizontal, F.Cu at (50.8, 92.4)
- added J11: TB007-508-03BE, TerminalBlock_CUI:TerminalBlock_CUI_TB007-508-03_1x03_P5.08mm_Horizontal, F.Cu at (76.1, 110.9)
- added J2: TB007-508-03BE, TerminalBlock_CUI:TerminalBlock_CUI_TB007-508-03_1x03_P5.08mm_Horizontal, F.Cu at (3.06, 5.42)
- added J3: TB007-508-03BE, TerminalBlock_CUI:TerminalBlock_CUI_TB007-508-03_1x03_P5.08mm_Horizontal, F.Cu at (3.06, 18.0)
- added J4: TB007-508-03BE, TerminalBlock_CUI:TerminalBlock_CUI_TB007-508-03_1x03_P5.08mm_Horizontal, F.Cu at (3.06, 30.6)
- added J5: TB007-508-03BE, TerminalBlock_CUI:TerminalBlock_CUI_TB007-508-03_1x03_P5.08mm_Horizontal, F.Cu at (3.06, 43.1)
- added J6: TB007-508-03BE, TerminalBlock_CUI:TerminalBlock_CUI_TB007-508-03_1x03_P5.08mm_Horizontal, F.Cu at (3.06, 55.7)
- added J7: TB007-508-03BE, TerminalBlock_CUI:TerminalBlock_CUI_TB007-508-03_1x03_P5.08mm_Horizontal, F.Cu at (3.06, 68.2)
- added J8: TB007-508-03BE, TerminalBlock_CUI:TerminalBlock_CUI_TB007-508-03_1x03_P5.08mm_Horizontal, F.Cu at (54.5, 60.8)
- added J9: TB007-508-03BE, TerminalBlock_CUI:TerminalBlock_CUI_TB007-508-03_1x03_P5.08mm_Horizontal, F.Cu at (49.0, 77.5)
- added U1: logic_level_conversor, level_shifter:CONV_BOB-12009_level_shifter, F.Cu at (76.3, 124.1)
